File: DXRP1.kicad_sch (KiCad schematic)
At the start: 49 parts, among them J1 USB_B_Micro, J11 5v, J12 VIN, J13 MB, J14 MA, J15 Servo 5V, J16 Servo signal, J17 Servo GND, J18 GND pad, J2 I2C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

Commit message: Revision 1.1
Added proper USB backpowering protection circuit
Parts:
- added Q1: AO3401A, Package_TO_SOT_SMD:SOT-23, symbol Transistor_FET:AO3401A
- added R2: 100k, Resistor_SMD:R_0603_1608Metric_Pad0.98x0.95mm_HandSolder, symbol Device:R
Connections:
- net +5V: now also Q1.3 (D); no longer C4.1, D1.1 (K), U3.1 (VIN), U3.3 (EN)
- net GND: now also R2.2
- net VUSB: now also Q1.1 (G), R2.1
- net VBUS renamed VMotor
- new net: C4.1, D1.1 (K), Q1.2 (S), U3.1 (VIN), U3.3 (EN)
Other:
- moved on the sheet: C4, C7, C9, D1, U3
